File: hardware/inputs.kicad_sch (KiCad schematic)
At the start: 16 parts, among them J12 JOY_L, J3 2x USB A, J5 2x USB A, J8 JOY_R, U10 74HC597, U14 74HC597, U15 FE1.1s, Y1 Crystal_GND24

Commit message: i2c expander
Parts:
- added D1, D2, D3, D4: LED, symbol Device:LED
- added R11, R45, R48, R9: 220, Resistor_SMD:R_0603_1608Metric_Pad0.98x0.95mm_HandSolder, symbol Device:R
- added SW5, SW6, SW7, SW8: SW_MEC_5G, symbol Switch:SW_MEC_5G
- added U17: MCP23008-xML, Package_DFN_QFN:QFN-20-1EP_4x4mm_P0.5mm_EP2.7x2.7mm, symbol Interface_Expansion:MCP23008-xML
- added U18: RP2040, Package_DFN_QFN:QFN-56-1EP_7x7mm_P0.4mm_EP3.2x3.2mm, symbol MCU_RaspberryPi:RP2040
Connections:
- net +3.3V: now also U17.18 (VDD), U17.4 (~{RESET})
- net GND: now also R11.1, R45.1, R48.1, R9.1, SW5.3 (B), SW5.4 (B), SW6.3 (B), SW6.4 (B), SW7.3 (B), SW7.4 (B), SW8.3 (B), SW8.4 (B), U17.1 (A2), U17.17 (VSS), U17.2 (A1), U17.3 (A0)
- net JOY_DATA: now reaches U14.9 (Q)
- new net: SW6.1 (A), SW6.2 (A), U17.10 (GP1)
- new net: D1.1 (K), U17.13 (GP4)
- new net: D1.2 (A), R9.2
- new net: D4.1 (K), U17.16 (GP7)
- new net: D4.2 (A), R48.2
- new net: SW8.1 (A), SW8.2 (A), U17.12 (GP3)
- new net: U18.1 (IOVDD), U18.10 (IOVDD), U18.22 (IOVDD), U18.33 (IOVDD), U18.42 (IOVDD), U18.49 (IOVDD)
- new net: U18.23 (DVDD), U18.50 (DVDD)
- new net: D2.1 (K), U17.14 (GP5)
- new net: D2.2 (A), R11.2
- new net: D3.1 (K), U17.15 (GP6)
- new net: D3.2 (A), R45.2
- new net: SW7.1 (A), SW7.2 (A), U17.11 (GP2)
- new net: SW5.1 (A), SW5.2 (A), U17.9 (GP0)
- new net I2C1_SCL: U17.19 (SCL)
- new net I2C1_SDA: U17.20 (SDA)
- no-connect marks 5 -> 6

Commit message: wip
Parts:
- removed C13, C14: 100n, Capacitor_SMD:C_0603_1608Metric_Pad1.08x0.95mm_HandSolder, symbol Device:C
- removed C28, C29: 10uF, symbol Device:C_Polarized
- removed D1, D2, D3, D4: LED, symbol Device:LED
- removed J3, J5: 2x USB A, symbol TRHMSX:2xUSB_A
- removed R11, R45, R48, R9: 220, Resistor_SMD:R_0603_1608Metric_Pad0.98x0.95mm_HandSolder, symbol Device:R
- removed R8: 2k7, Resistor_SMD:R_0603_1608Metric_Pad0.98x0.95mm_HandSolder, symbol Device:R
- removed SW5, SW6, SW7, SW8: SW_MEC_5G, symbol Switch:SW_MEC_5G
- removed U15: FE1.1s, Package_SO:SSOP-28_3.9x9.9mm_P0.635mm, symbol Interface_USB:FE1.1s
- removed U17: MCP23008-xML, Package_DFN_QFN:QFN-20-1EP_4x4mm_P0.5mm_EP2.7x2.7mm, symbol Interface_Expansion:MCP23008-xML
- removed U18: RP2040, Package_DFN_QFN:QFN-56-1EP_7x7mm_P0.4mm_EP3.2x3.2mm, symbol MCU_RaspberryPi:RP2040
- removed Y1: Crystal_GND24, symbol Device:Crystal_GND24
- added C47, C48: 100n, Capacitor_SMD:C_0603_1608Metric_Pad1.08x0.95mm_HandSolder, symbol Device:C
- added J10: JOY_2, symbol Connector:DE9_Socket_MountingHoles
- added J15: JOY_3, symbol Connector:DE9_Socket_MountingHoles
- added JP1, JP2: SolderJumper, symbol Jumper:SolderJumper_3_Open
- added R28, R37, R38: 33R, symbol Device:R
- added R35: 10K, symbol Device:R
- added RN12, RN13, RN14, RN15, RN16, RN19: 10K, symbol Device:R_Pack04
- added U15, U4: 74HC597, symbol Chimera:74HC597
- added U23: 25CS320, Package_SO:SOIC-8_3.9x4.9mm_P1.27mm, symbol TRHMSX:25CS320
- J12: value JOY_L -> JOY_1
- J8: value JOY_R -> JOY_0
- U10, U14: symbol TRHMSX:74HC597 -> Chimera:74HC597
Connections:
- net +3.3V: now also C11.1, U10.10 (~{MR}), U10.14 (DS), U14.10 (~{MR}), C47.2, C48.2, R35.2, U15.10 (~{MR}), U15.16 (VCC), U23.8 (V_{CC}), U4.10 (~{MR}), U4.16 (VCC)
- net +5V: now also J12.5, J8.5, J10.5, J15.5, RN12.5 (R4.2), RN12.6 (R3.2), RN12.7 (R2.2), RN12.8 (R1.2), RN13.5 (R4.2), RN13.6 (R3.2), RN13.7 (R2.2), RN13.8 (R1.2), RN14.1 (R1.1), RN14.2 (R2.1), RN14.3 (R3.1), RN14.4 (R4.1), RN15.5 (R4.2), RN15.6 (R3.2), RN15.7 (R2.2), RN15.8 (R1.2), RN16.1 (R1.1), RN16.2 (R2.1), RN16.3 (R3.1), RN16.4 (R4.1), RN19.5 (R4.2), RN19.6 (R3.2), RN19.7 (R2.2), RN19.8 (R1.2)
- net GND: now also J12.8, J8.8, C47.1, C48.1, J10.0 (PAD), J10.8, J15.0 (PAD), J15.8, U15.8 (GND), U23.4 (V_{SS}), U4.8 (GND)
- net at U10.1 (D1): now also J8.6, RN12.2 (R2.1)
- net CTLB_SCK: now reaches U10.11 (SHCP)
- net CTLB_SCK: now also U14.11 (SHCP), U15.11 (SHCP), U23.6 (SCK), U4.11 (SHCP)
- net CTLB_J_LOAD: now reaches U10.13 (~{PL})
- net CTLB_J_LOAD: now also U14.13 (~{PL}), U15.13 (~{PL}), U4.13 (~{PL})
- net at J8.1, U10.15 (D0): now also RN12.1 (R1.1)
- net at U10.2 (D2): now also J8.2, RN12.3 (R3.1)
- net at U10.3 (D3): now also J8.3, RN12.4 (R4.1)
- net at U10.4 (D4): now also J8.4, RN13.2 (R2.1)
- net at U10.5 (D5): now also J8.9, RN13.1 (R1.1)
- net at U14.1 (D1): now also J12.6, RN13.4 (R4.1)
- net at J12.1, U14.15 (D0): now also RN13.3 (R3.1)
- net at U14.2 (D2): now also J12.2, RN14.5 (R4.2)
- net at U14.3 (D3): now also J12.3, RN14.6 (R3.2)
- net at U14.4 (D4): now also J12.4, RN14.7 (R2.2)
- net at U14.5 (D5): now also J12.9, RN14.8 (R1.2)
- net CTLB_J_CS: now reaches J12.7
- net CTLB_J_CS: now also J8.7, J10.7, J15.7
- net JOY_DATA: no longer names the net of U14.9 (Q)
- net JOY_DATA: now also JP1.2 (C)
- new net: J10.9, RN19.1 (R1.1), U4.5 (D5)
- new net: J10.4, RN19.2 (R2.1), U4.4 (D4)
- new net: J15.1, RN19.3 (R3.1), U15.15 (D0)
- new net: J15.6, RN19.4 (R4.1), U15.1 (D1)
- new net: JP2.1 (A), R38.1
- new net: JP2.2 (C), U4.9 (Q)
- new net: JP2.3 (B), U15.14 (DS)
- new net: J10.1, RN15.1 (R1.1), U4.15 (D0)
- new net: J10.2, RN15.3 (R3.1), U4.2 (D2)
- new net: J10.3, RN15.4 (R4.1), U4.3 (D3)
- new net: J10.6, RN15.2 (R2.1), U4.1 (D1)
- new net: JP1.1 (A), R37.1
- new net: J15.9, RN16.5 (R4.2), U15.5 (D5)
- new net: J15.4, RN16.6 (R3.2), U15.4 (D4)
- new net: J15.3, RN16.7 (R2.2), U15.3 (D3)
- new net: J15.2, RN16.8 (R1.2), U15.2 (D2)
- new net: R28.2, U23.2 (SO)
- new net: JP1.3 (B), U4.14 (DS)
- new net CTLB_CF_CS: R35.1, U23.1 (~{CS})
- new net CTLB_J_LATCH: U10.12 (STCP), U14.12 (STCP), U15.12 (STCP), U4.12 (STCP)
- new net CTLB_SI(MOSI): U23.5 (SI)
- new net CTLB_SO(MISO): R28.1, R37.2, R38.2, U15.9 (Q)
- no-connect marks 6 -> 0
Other:
- moved on the sheet: C1, C9, J12, J8, U10, U14
