File: hardware/msxxx.kicad_sch (KiCad schematic)
At the start: 106 parts, among them IC4 NC7WZU04P6X, IC8 EPCS4, J10 JOY2, J11 USB_C_Receptacle_PowerOnly_6P, J15 JOY1, J17 Conn_01x02, J2 Conn_02x04_Odd_Even, J4 Micro_SD_Card_Det1, J6 USB_A, J7 Mini-DIN-6, J8 Conn_02x05_Odd_Even, J9 Conn_02x25_Odd_Even, Q1 AO3400A, SW2 SW_Push, SW3 SW_Push, U1 EP1C12Q240C8N, U10 74HC4066D_653, U2 AMS1117-1.5, U3 AMS1117-3.3, U5 MT48LC16M16A2TG, U6 M51953BFP, U7 CH559T, U8 IP2721, U9 74HC4066D_653, Y1 Crystal

Commit message: wip
Parts:
- C10, C11, C12, C13, C14, C15, C16, C17, C18, C19, C2, C20, C21, C22, C23, C24, C25, C3, C33, C34, C35, C4, C55, C56, C6, C7, C9: footprint Capacitor_SMD:C_0805_2012Metric -> Capacitor_SMD:C_0603_1608Metric_Pad1.08x0.95mm_HandSolder
- IC4: footprint SOT65P210X110-6N -> (none)
- R1, R10, R11, R12, R13, R14, R2, R3, R5, R7, R8, R9: footprint Resistor_SMD:R_0805_2012Metric -> Resistor_SMD:R_0603_1608Metric_Pad0.98x0.95mm_HandSolder
- U1: footprint QFP50P3460X3460X410-240N -> Package_QFP:PQFP-240_32.1x32.1mm_P0.5mm
Changed lines of the file:
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@@
 			)
 		)
-		(property "Footprint" "Capacitor_SMD:C_0805_2012Metric"
+		(property "Footprint" "Capacitor_SMD:C_0603_1608Metric_Pad1.08x0.95mm_HandSolder"
 			(at 136.1948 54.61 0)
 			(effects
@@
 			)
 		)
-		(property "Footprint" "Resistor_SMD:R_0805_2012Metric"
+		(property "Footprint" "Resistor_SMD:R_0603_1608Metric_Pad0.98x0.95mm_HandSolder"
 			(at 328.93 92.202 90)
 			(effects
@@
 			)
 		)
-		(property "Footprint" "Capacitor_SMD:C_0805_2012Metric"
+		(property "Footprint" "Capacitor_SMD:C_0603_1608Metric_Pad1.08x0.95mm_HandSolder"
 			(at 384.5052 276.86 0)
 			(effects
@@
 			)
 		)
-		(property "Footprint" "Resistor_SMD:R_0805_2012Metric"
+		(property "Footprint" "Resistor_SMD:R_0603_1608Metric_Pad0.98x0.95mm_HandSolder"
 			(at 306.07 372.872 90)
 			(effects
@@
 			)
 		)
-		(property "Footprint" "Capacitor_SMD:C_0805_2012Metric"
+		(property "Footprint" "Capacitor_SMD:C_0603_1608Metric_Pad1.08x0.95mm_HandSolder"
 			(at 257.5052 389.89 0)
 			(effects
@@
 			)
 		)
-		(property "Footprint" "Capacitor_SMD:C_0805_2012Metric"
+		(property "Footprint" "Capacitor_SMD:C_0603_1608Metric_Pad1.08x0.95mm_HandSolder"
 			(at 194.0052 389.89 0)
 			(effects
@@
 			)
 		)
-		(property "Footprint" "Capacitor_SMD:C_0805_2012Metric"
+		(property "Footprint" "Capacitor_SMD:C_0603_1608Metric_Pad1.08x0.95mm_HandSolder"
 			(at 319.7352 393.7 0)
 			(effects
@@
 			)
 		)
-		(property "Footprint" "Capacitor_SMD:C_0805_2012Metric"
+		(property "Footprint" "Capacitor_SMD:C_0603_1608Metric_Pad1.08x0.95mm_HandSolder"
 			(at 145.7452 396.24 0)
 			(effects
@@
 			)
 		)
-		(property "Footprint" "Capacitor_SMD:C_0805_2012Metric"
+		(property "Footprint" "Capacitor_SMD:C_0603_1608Metric_Pad1.08x0.95mm_HandSolder"
 			(at 425.1452 309.88 0)
 			(effects
@@
 			)
 		)
-		(property "Footprint" "Capacitor_SMD:C_0805_2012Metric"
+		(property "Footprint" "Capacitor_SMD:C_0603_1608Metric_Pad1.08x0.95mm_HandSolder"
 			(at 420.0652 379.73 0)
 			(effects
@@
 			)
 		)
-		(property "Footprint" "Resistor_SMD:R_0805_2012Metric"
+		(property "Footprint" "Resistor_SMD:R_0603_1608Metric_Pad0.98x0.95mm_HandSolder"
 			(at 219.202 317.5 90)
 			(effects
@@
 			)
 		)
-		(property "Footprint" "Resistor_SMD:R_0805_2012Metric"
+		(property "Footprint" "Resistor_SMD:R_0603_1608Metric_Pad0.98x0.95mm_HandSolder"
 			(at 151.13 62.992 90)
 			(effects
@@
 			)
 		)
-		(property "Footprint" "Resistor_SMD:R_0805_2012Metric"
+		(property "Footprint" "Resistor_SMD:R_0603_1608Metric_Pad0.98x0.95mm_HandSolder"
 			(at 207.772 317.5 90)
 			(effects
@@
 			)
 		)
-		(property "Footprint" "Capacitor_SMD:C_0805_2012Metric"
+		(property "Footprint" "Capacitor_SMD:C_0603_1608Metric_Pad1.08x0.95mm_HandSolder"
 			(at 386.08 40.9448 0)
 			(effects
@@
 			)
 		)
-		(property "Footprint" "Capacitor_SMD:C_0805_2012Metric"
+		(property "Footprint" "Capacitor_SMD:C_0603_1608Metric_Pad1.08x0.95mm_HandSolder"
 			(at 160.9852 389.89 0)
 			(effects
@@
 			)
 		)
-		(property "Footprint" "Resistor_SMD:R_0805_2012Metric"
+		(property "Footprint" "Resistor_SMD:R_0603_1608Metric_Pad0.98x0.95mm_HandSolder"
 			(at 309.372 260.35 90)
 			(effects
@@
 			)
 		)
-		(property "Footprint" "Resistor_SMD:R_0805_2012Metric"
+		(property "Footprint" "Resistor_SMD:R_0603_1608Metric_Pad0.98x0.95mm_HandSolder"
 			(at 270.51 49.022 90)
 			(effects
@@
 			)
 		)
-		(property "Footprint" "Capacitor_SMD:C_0805_2012Metric"
+		(property "Footprint" "Capacitor_SMD:C_0603_1608Metric_Pad1.08x0.95mm_HandSolder"
 			(at 380.6952 323.85 0)
 			(effects
@@
 			)
 		)
-		(property "Footprint" "Capacitor_SMD:C_0805_2012Metric"
+		(property "Footprint" "Capacitor_SMD:C_0603_1608Metric_Pad1.08x0.95mm_HandSolder"
 			(at 395.9352 276.86 0)
 			(effects
@@
 			)
 		)
-		(property "Footprint" "QFP50P3460X3460X410-240N"
+		(property "Footprint" "Package_QFP:PQFP-240_32.1x32.1mm_P0.5mm"
 			(at 67.31 109.22 0)
 			(effects
@@
 			)
 		)
-		(property "Footprint" "Capacitor_SMD:C_0805_2012Metric"
+		(property "Footprint" "Capacitor_SMD:C_0603_1608Metric_Pad1.08x0.95mm_HandSolder"
 			(at 386.08 26.9748 0)
 			(effects
@@
 			)
 		)
-		(property "Footprint" "QFP50P3460X3460X410-240N"
+		(property "Footprint" "Package_QFP:PQFP-240_32.1x32.1mm_P0.5mm"
 			(at 298.45 106.68 0)
 			(effects
@@
 			)
 		)
-		(property "Footprint" "Resistor_SMD:R_0805_2012Metric"
+		(property "Footprint" "Resistor_SMD:R_0603_1608Metric_Pad0.98x0.95mm_HandSolder"
 			(at 306.07 381.762 90)
 			(effects
@@
 			)
 		)
-		(property "Footprint" "Capacitor_SMD:C_0805_2012Metric"
+		(property "Footprint" "Capacitor_SMD:C_0603_1608Metric_Pad1.08x0.95mm_HandSolder"
 			(at 224.4852 389.89 0)
 			(effects
@@
 			)
 		)
-		(property "Footprint" "Resistor_SMD:R_0805_2012Metric"
+		(property "Footprint" "Resistor_SMD:R_0603_1608Metric_Pad0.98x0.95mm_HandSolder"
 			(at 106.68 362.458 90)
 			(effects
@@
 			)
 		)
-		(property "Footprint" "Resistor_SMD:R_0805_2012Metric"
+		(property "Footprint" "Resistor_SMD:R_0603_1608Metric_Pad0.98x0.95mm_HandSolder"
 			(at 374.65 296.672 90)
 			(effects
@@
 			)
 		)
-		(property "Footprint" "Capacitor_SMD:C_0805_2012Metric"
+		(property "Footprint" "Capacitor_SMD:C_0603_1608Metric_Pad1.08x0.95mm_HandSolder"
 			(at 386.08 113.3348 0)
 			(effects
@@
 			)
 		)
-		(property "Footprint" "Capacitor_SMD:C_0805_2012Metric"
+		(property "Footprint" "Capacitor_SMD:C_0603_1608Metric_Pad1.08x0.95mm_HandSolder"
 			(at 372.11 395.2748 0)
 			(effects
@@
 			)
 		)
-		(property "Footprint" "Resistor_SMD:R_0805_2012Metric"
+		(property "Footprint" "Resistor_SMD:R_0603_1608Metric_Pad0.98x0.95mm_HandSolder"
 			(at 357.378 381 90)
 			(effects
@@
 			)
 		)
-		(property "Footprint" "QFP50P3460X3460X410-240N"
+		(property "Footprint" "Package_QFP:PQFP-240_32.1x32.1mm_P0.5mm"
 			(at 185.42 102.87 0)
 			(effects
@@
 			)
 		)
-		(property "Footprint" "Capacitor_SMD:C_0805_2012Metric"
+		(property "Footprint" "Capacitor_SMD:C_0603_1608Metric_Pad1.08x0.95mm_HandSolder"
 			(at 253.6952 63.5 0)
 			(effects
@@
 			)
 		)
-		(property "Footprint" "Capacitor_SMD:C_0805_2012Metric"
+		(property "Footprint" "Capacitor_SMD:C_0603_1608Metric_Pad1.08x0.95mm_HandSolder"
 			(at 386.08 63.8048 0)
 			(effects
@@
 			)
 		)
-		(property "Footprint" "Capacitor_SMD:C_0805_2012Metric"
+		(property "Footprint" "Capacitor_SMD:C_0603_1608Metric_Pad1.08x0.95mm_HandSolder"
 			(at 386.08 98.0948 0)
 			(effects
@@
 			)
 		)
-		(property "Footprint" "Capacitor_SMD:C_0805_2012Metric"
+		(property "Footprint" "Capacitor_SMD:C_0603_1608Metric_Pad1.08x0.95mm_HandSolder"
 			(at 122.8852 396.24 0)
 			(effects
@@
 			)
 		)
-		(property "Footprint" "Capacitor_SMD:C_0805_2012Metric"
+		(property "Footprint" "Capacitor_SMD:C_0603_1608Metric_Pad1.08x0.95mm_HandSolder"
 			(at 386.08 126.0348 0)
 			(effects
@@
 			)
 		)
-		(property "Footprint" "Capacitor_SMD:C_0805_2012Metric"
+		(property "Footprint" "Capacitor_SMD:C_0603_1608Metric_Pad1.08x0.95mm_HandSolder"
 			(at 523.24 341.3252 0)
 			(effects
@@
 			)
 		)
-		(property "Footprint" "Capacitor_SMD:C_0805_2012Metric"
+		(property "Footprint" "Capacitor_SMD:C_0603_1608Metric_Pad1.08x0.95mm_HandSolder"
 			(at 386.08 140.0048 0)
 			(effects
@@
 			)
 		)
-		(property "Footprint" "SOT65P210X110-6N"
+		(property "Footprint" ""
 			(at 326.39 288.62 0)
 			(effects
@@
 			)
 		)
-		(property "Footprint" "Resistor_SMD:R_0805_2012Metric"
+		(property "Footprint" "Resistor_SMD:R_0603_1608Metric_Pad0.98x0.95mm_HandSolder"
 			(at 309.118 260.35 90)
 			(effects
@@
 			)
 		)
-		(property "Footprint" "Capacitor_SMD:C_0805_2012Metric"
+		(property "Footprint" "Capacitor_SMD:C_0603_1608Metric_Pad1.08x0.95mm_HandSolder"
 			(at 562.61 253.0348 0)
 			(effects
@@
 			)
 		)
-		(property "Footprint" "Capacitor_SMD:C_0805_2012Metric"
+		(property "Footprint" "Capacitor_SMD:C_0603_1608Metric_Pad1.08x0.95mm_HandSolder"
 			(at 445.4652 397.51 0)
 			(effects
@@
 			)
 		)
-		(property "Footprint" "Capacitor_SMD:C_0805_2012Metric"
+		(property "Footprint" "Capacitor_SMD:C_0603_1608Metric_Pad1.08x0.95mm_HandSolder"
 			(at 372.11 368.6048 0)
 			(effects
@@
 			)
 		)
-		(property "Footprint" "Capacitor_SMD:C_0805_2012Metric"
+		(property "Footprint" "Capacitor_SMD:C_0603_1608Metric_Pad1.08x0.95mm_HandSolder"
 			(at 386.08 52.3748 0)
 			(effects

Commit message: pico led and buttons, virtual leds
Parts:
- removed C28, C29: C_Polarized, Capacitor_SMD:CP_Elec_6.3x3, symbol Device:C_Polarized
- removed C9: C, Capacitor_SMD:C_0603_1608Metric_Pad1.08x0.95mm_HandSolder, symbol Device:C
- removed IC8: EPCS4, EPCS4:SO08, symbol TRHMSX:EPCS4
- removed J8: Conn_02x05_Odd_Even, Connector_PinHeader_2.54mm:PinHeader_2x05_P2.54mm_Vertical, symbol Connector_Generic:Conn_02x05_Odd_Even
- removed RN12, RN17, RN18, RN19, RN20, RN27, RN28, RN29, RN36, RN37, RN38: R_Pack04_Split, Resistor_SMD:R_Array_Convex_4x0603, symbol Device:R_Pack04_Split
- removed unit 3 of RN16
- removed unit 4 of RN16
- removed U10, U9: 74HC4066D_653, 74HC4066D_653:SOIC127P600X175-14N, symbol 74HC4066D_653:74HC4066D_653
- added SW1, SW2, SW3, SW4: SW_MEC_5G, symbol Switch:SW_MEC_5G
- added U9: ~, TRHMSX:SSD1306-0.91-OLED-4pin-128x32, symbol TRHMSX:Display_OLED_I2C
Connections:
- net +3.3V: now also U1.35 (MSEL1)
- net AS_CK: now also A1.24 (GPIO18)
- net AS_DI: now also A1.25 (GPIO19)
- net C_CONF: now also A1.21 (GPIO16)
- net C_DONE: now also A1.26 (GPIO20)
- net C_STAT: now also A1.22 (GPIO17)
- net GND: now also SW1.3 (B), SW1.4 (B), SW2.3 (B), SW2.4 (B), SW3.3 (B), SW3.4 (B), SW4.3 (B), SW4.4 (B), U9.1 (GND); no longer U1.35 (MSEL1)
- net at A1.14 (GPIO10): now also SW1.1 (A), SW1.2 (A)
- net at A1.15 (GPIO11): now also SW2.1 (A), SW2.2 (A)
- net at A1.16 (GPIO12): now also SW3.1 (A), SW3.2 (A)
- net at A1.17 (GPIO13): now also SW4.1 (A), SW4.2 (A)
- net C_CS: now reaches A1.27 (GPIO21)
- net at A1.36 (3V3): now also U9.2 (VCC)
- net at A1.4 (GPIO2): now also U9.4 (SDA)
- net at A1.5 (GPIO3): now also U9.3 (SCL)
- no-connect marks 35 -> 47

Commit message: pico test firmware
Parts:
- removed C11, C13, C14: C, Capacitor_SMD:C_0603_1608Metric_Pad1.08x0.95mm_HandSolder, symbol Device:C
- removed IC4: NC7WZU04P6X, symbol TRHMSX:NC7WZU04P6X
- removed R11, R8, R9: R, Resistor_SMD:R_0603_1608Metric_Pad0.98x0.95mm_HandSolder, symbol Device:R
- removed Y1: Crystal, Crystal:Crystal_HC49-U_Vertical, symbol Device:Crystal
- added R46, R47: 100, Resistor_SMD:R_0603_1608Metric_Pad0.98x0.95mm_HandSolder, symbol Device:R
- added Y2: 21.47727 MHz, Oscillator:Oscillator_SMD_SeikoEpson_SG8002CA-4Pin_7.0x5.0mm, symbol Oscillator:SG-7050CCN
- J2: value Conn_02x04_Odd_Even -> ESP-01
- R7: value R -> 10
Connections:
- net +3.3V: now also Y2.4 (Vcc)
- net CLK21M: now also R46.2, R47.2, Y2.3 (OUT); no longer U1.28 (CLK0)
- net PWRLED: now also A1.20 (GPIO15); no longer U1.240 (IO)
- net EXTCLK: no longer names the net of U1.29 (CLK1)
- net EXTCLK: now also R47.1
- new net: Y2.1 (OE), Y2.2 (GND)
- new net: R46.1, U1.28 (CLK0)
- no-connect marks 47 -> 48
Other:
- moved on the sheet: C10, J4, J9, R1, R2, R7, SW1, SW2, SW3, SW4, U9

Commit message: wip
Connections:
- net at A1.4 (GPIO2): no longer U9.4 (SDA)
- net at A1.5 (GPIO3): no longer U9.3 (SCL)
- net at A1.6 (GPIO4): now also U9.4 (SDA)
- net at A1.7 (GPIO5): now also U9.3 (SCL)
Other:
- added sheet inputs (inputs.kicad_sch)
Changed lines of the file:
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@@
 	(wire
 		(pts
-			(xy 96.52 248.92) (xy 101.6 248.92)
+			(xy 96.52 243.84) (xy 101.6 243.84)
 		)
 		(stroke
@@
 	(wire
 		(pts
-			(xy 101.6 269.24) (xy 101.6 248.92)
+			(xy 101.6 269.24) (xy 101.6 243.84)
 		)
 		(stroke
@@
 	(wire
 		(pts
+			(xy 96.52 246.38) (xy 104.14 246.38)
+		)
+		(stroke
+			(width 0)
+			(type default)
+		)
+	)
+	(wire
+		(pts
 			(xy 340.36 162.56) (xy 345.44 162.56)
 		)
@@
 	(wire
 		(pts
-			(xy 104.14 266.7) (xy 104.14 251.46)
+			(xy 104.14 266.7) (xy 104.14 246.38)
 		)
 		(stroke
@@
 	(wire
 		(pts
-			(xy 96.52 251.46) (xy 104.14 251.46)
-		)
-		(stroke
-			(width 0)
-			(type default)
-		)
-	)
-	(wire
-		(pts
 			(xy 575.31 340.36) (xy 542.29 340.36)
 		)
@@
 				)
 			)
+		)
+	)
+	(sheet
+		(at 393.7 431.8)
+		(size 114.3 74.93)
+		(exclude_from_sim no)
+		(in_bom yes)
+		(on_board yes)
+		(dnp no)
+		(fields_autoplaced yes)
+		(stroke
+			(width 0.1524)
+			(type solid)
+		)
+		(fill
+			(color 0 0 0 0.0000)
+		)
+		(property "Sheetname" "inputs"
+			(at 393.7 431.0884 0)
+			(effects
+				(font
+					(size 1.27 1.27)
+				)
+				(justify left bottom)
+			)
+		)
+		(property "Sheetfile" "inputs.kicad_sch"
+			(at 393.7 507.3146 0)
+			(effects
+				(font
+					(size 1.27 1.27)
+				)
+				(justify left top)
+			)
+		)
+		(instances
+			(project "msxxx"
+				(path "/9009b6ae-d2e5-4e55-a5ae-61e06cafcec3"
+					(page "5")
+				)
+			)

Commit message: wip
Parts:
- removed A1: RaspberryPi_Pico, Module:RaspberryPi_Pico_Common_Unspecified, symbol MCU_Module:RaspberryPi_Pico
- removed C10, C12, C15, C16, C17, C18, C19, C2, C20, C21, C22, C23, C24, C25, C3, C33, C34, C35, C4, C6, C7: C, Capacitor_SMD:C_0603_1608Metric_Pad1.08x0.95mm_HandSolder, symbol Device:C
- removed C5, C8: C_Polarized, Capacitor_SMD:CP_Elec_6.3x3, symbol Device:C_Polarized
- removed C55: 10uF, Capacitor_SMD:C_0603_1608Metric_Pad1.08x0.95mm_HandSolder, symbol Device:C
- removed C56: 1uF, Capacitor_SMD:C_0603_1608Metric_Pad1.08x0.95mm_HandSolder, symbol Device:C
- removed D10, D9: LED, LED_SMD:LED_0805_2012Metric, symbol Device:LED
- removed J10: JOY2, Connector_Dsub:DSUB-9_Male_Horizontal_P2.77x2.84mm_EdgePinOffset4.94mm_Housed_MountingHolesOffset7.48mm, symbol Connector:DE9_Plug
- removed J11: USB_C_Receptacle_PowerOnly_6P, Connector_USB:USB_C_Receptacle_GCT_USB4125-xx-x-0190_6P_TopMnt_Horizontal, symbol Connector:USB_C_Receptacle_PowerOnly_6P
- removed J15: JOY1, Connector_Dsub:DSUB-9_Male_Horizontal_P2.77x2.84mm_EdgePinOffset4.94mm_Housed_MountingHolesOffset7.48mm, symbol Connector:DE9_Plug
- removed J17: Conn_01x02, Connector_PinHeader_2.54mm:PinHeader_1x02_P2.54mm_Vertical, symbol Connector_Generic:Conn_01x02
- removed J2: ESP-01, Connector_PinSocket_2.54mm:PinSocket_2x04_P2.54mm_Vertical, symbol Connector_Generic:Conn_02x04_Odd_Even
- removed J4: Micro_SD_Card_Det1, CRISAG:Conn_uSDcard, symbol TRHMSX:Micro_SD_Card_Det1
- removed J6: USB_A, TRHMSX:TE_6364372-2, symbol Connector:USB_A
- removed J7: Mini-DIN-6, TRHMSX:TE_5749180-1, symbol Connector:Mini-DIN-6
- removed J9: Conn_02x25_Odd_Even, Connector_PinHeader_2.54mm:PinHeader_2x25_P2.54mm_Vertical, symbol Connector_Generic:Conn_02x25_Odd_Even
- removed Q1: AO3400A, Package_TO_SOT_SMD:SOT-23, symbol Transistor_FET:AO3400A
- removed R1, R10, R12, R13, R14, R2, R3, R5: R, Resistor_SMD:R_0603_1608Metric_Pad0.98x0.95mm_HandSolder, symbol Device:R
- removed R43, R44: 5k1, Resistor_SMD:R_0603_1608Metric_Pad0.98x0.95mm_HandSolder, symbol Device:R
- removed R46, R47: 100, Resistor_SMD:R_0603_1608Metric_Pad0.98x0.95mm_HandSolder, symbol Device:R
- removed R7: 10, Resistor_SMD:R_0603_1608Metric_Pad0.98x0.95mm_HandSolder, symbol Device:R
- removed RN1, RN10, RN11, RN13, RN14, RN15, RN16, RN2, RN21, RN22, RN23, RN25, RN26, RN3, RN35, RN4, RN44, RN5, RN6, RN7, RN8, RN9: R_Pack04_Split, Resistor_SMD:R_Array_Convex_4x0603, symbol Device:R_Pack04_Split
- removed SW1, SW2, SW3, SW4: SW_MEC_5G, symbol Switch:SW_MEC_5G
- removed SW2: SW_Push, Button_Switch_THT:SW_Tactile_SPST_Angled_PTS645Vx83-2LFS, symbol Switch:SW_Push
- removed SW3: SW_Push, Button_Switch_SMD:SW_Push_1P1T_NO_6x6mm_H9.5mm, symbol Switch:SW_Push
- removed U1: EP1C12Q240C8N, Package_QFP:PQFP-240_32.1x32.1mm_P0.5mm, symbol TRHMSX:EP1C12Q240C8N
- removed U2: AMS1117-1.5, Package_TO_SOT_SMD:SOT-223-3_TabPin2, symbol Regulator_Linear:AMS1117-1.5
- removed U3: AMS1117-3.3, Package_TO_SOT_SMD:SOT-223-3_TabPin2, symbol Regulator_Linear:AMS1117-3.3
- removed U5: MT48LC16M16A2TG, Package_SO:TSOP-II-54_22.2x10.16mm_P0.8mm, symbol Memory_RAM:MT48LC16M16A2TG
- removed U6: M51953BFP, TRHMSX:SO08, symbol TRHMSX:M51953BFP
- removed U7: CH559T, Package_SO:SSOP-20_5.3x7.2mm_P0.65mm, symbol CH55x:CH559T
- removed U8: IP2721, Package_SO:TSSOP-16_4.4x5mm_P0.65mm, symbol Interface_USB:IP2721
- removed U9: ~, TRHMSX:SSD1306-0.91-OLED-4pin-128x32, symbol TRHMSX:Display_OLED_I2C
- removed Y2: 21.47727 MHz, Oscillator:Oscillator_SMD_SeikoEpson_SG8002CA-4Pin_7.0x5.0mm, symbol Oscillator:SG-7050CCN
Connections:
- no-connect marks 48 -> 0
Other:
- sheet audio renamed misc
- sheet inputs renamed controllers_board
- sheet slots renamed platfrom_io
- sheet video renamed av
- added sheet controller_board_n64 (controller_board_n64/controller_board_n64/controller_board_n64.kicad_sch)
- added sheet main (main.kicad_sch)
- company: The Retro Hacker -> Good
- title: TRHMSX - A simple MSX2+ clone in FPGA -> FPGA retro platform
