File: hardware/video.kicad_sch (KiCad schematic)
At the start: 35 parts, among them J1 DH15, J13 MD-40SM, J16 Conn_Coaxial, U11 AD725, U12 ADV7123, U13 AD8073JNZ, X1 SCART-F

Commit message: wip
Parts:
- C27, C32, C37, C38, C39, C43, C44: footprint Capacitor_SMD:C_0805_2012Metric -> Capacitor_SMD:C_0603_1608Metric_Pad1.08x0.95mm_HandSolder
- R15, R16, R17, R18, R19, R20, R21, R22, R23, R24, R25, R26, R27, R28, R4, R6: footprint Resistor_SMD:R_0805_2012Metric -> Resistor_SMD:R_0603_1608Metric_Pad0.98x0.95mm_HandSolder
- X1: footprint SCART-F:SCART-F -> TRHMSX:SCART-F
Changed lines of the file:
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@@
 			)
 		)
-		(property "Footprint" "Capacitor_SMD:C_0805_2012Metric"
+		(property "Footprint" "Capacitor_SMD:C_0603_1608Metric_Pad1.08x0.95mm_HandSolder"
 			(at 163.83 146.3548 0)
 			(effects
@@
 			)
 		)
-		(property "Footprint" "Capacitor_SMD:C_0805_2012Metric"
+		(property "Footprint" "Capacitor_SMD:C_0603_1608Metric_Pad1.08x0.95mm_HandSolder"
 			(at 214.3252 121.92 0)
 			(effects
@@
 			)
 		)
-		(property "Footprint" "Resistor_SMD:R_0805_2012Metric"
+		(property "Footprint" "Resistor_SMD:R_0603_1608Metric_Pad0.98x0.95mm_HandSolder"
 			(at 85.09 205.232 90)
 			(effects
@@
 			)
 		)
-		(property "Footprint" "Resistor_SMD:R_0805_2012Metric"
+		(property "Footprint" "Resistor_SMD:R_0603_1608Metric_Pad0.98x0.95mm_HandSolder"
 			(at 175.768 187.96 90)
 			(effects
@@
 			)
 		)
-		(property "Footprint" "Resistor_SMD:R_0805_2012Metric"
+		(property "Footprint" "Resistor_SMD:R_0603_1608Metric_Pad0.98x0.95mm_HandSolder"
 			(at 208.28 192.532 90)
 			(effects
@@
 			)
 		)
-		(property "Footprint" "Resistor_SMD:R_0805_2012Metric"
+		(property "Footprint" "Resistor_SMD:R_0603_1608Metric_Pad0.98x0.95mm_HandSolder"
 			(at 264.16 141.732 90)
 			(effects
@@
 			)
 		)
-		(property "Footprint" "Capacitor_SMD:C_0805_2012Metric"
+		(property "Footprint" "Capacitor_SMD:C_0603_1608Metric_Pad1.08x0.95mm_HandSolder"
 			(at 148.59 151.4348 0)
 			(effects
@@
 			)
 		)
-		(property "Footprint" "Capacitor_SMD:C_0805_2012Metric"
+		(property "Footprint" "Capacitor_SMD:C_0603_1608Metric_Pad1.08x0.95mm_HandSolder"
 			(at 125.4252 240.03 0)
 			(effects
@@
 			)
 		)
-		(property "Footprint" "Resistor_SMD:R_0805_2012Metric"
+		(property "Footprint" "Resistor_SMD:R_0603_1608Metric_Pad0.98x0.95mm_HandSolder"
 			(at 81.28 150.368 90)
 			(effects
@@
 			)
 		)
-		(property "Footprint" "Capacitor_SMD:C_0805_2012Metric"
+		(property "Footprint" "Capacitor_SMD:C_0603_1608Metric_Pad1.08x0.95mm_HandSolder"
 			(at 186.3852 121.92 0)
 			(effects
@@
 			)
 		)
-		(property "Footprint" "Resistor_SMD:R_0805_2012Metric"
+		(property "Footprint" "Resistor_SMD:R_0603_1608Metric_Pad0.98x0.95mm_HandSolder"
 			(at 208.28 182.372 90)
 			(effects
@@
 			)
 		)
-		(property "Footprint" "Capacitor_SMD:C_0805_2012Metric"
+		(property "Footprint" "Capacitor_SMD:C_0603_1608Metric_Pad1.08x0.95mm_HandSolder"
 			(at 156.21 148.8948 0)
 			(effects
@@
 			)
 		)
-		(property "Footprint" "Capacitor_SMD:C_0805_2012Metric"
+		(property "Footprint" "Capacitor_SMD:C_0603_1608Metric_Pad1.08x0.95mm_HandSolder"
 			(at 106.3752 199.39 0)
 			(effects
@@
 			)
 		)
-		(property "Footprint" "SCART-F:SCART-F"
+		(property "Footprint" "TRHMSX:SCART-F"
 			(at 224.79 194.31 0)
 			(effects
@@
 			)
 		)
-		(property "Footprint" "Resistor_SMD:R_0805_2012Metric"
+		(property "Footprint" "Resistor_SMD:R_0603_1608Metric_Pad0.98x0.95mm_HandSolder"
 			(at 193.548 193.04 90)
 			(effects
@@
 			)
 		)
-		(property "Footprint" "Resistor_SMD:R_0805_2012Metric"
+		(property "Footprint" "Resistor_SMD:R_0603_1608Metric_Pad0.98x0.95mm_HandSolder"
 			(at 100.33 215.392 90)
 			(effects
@@
 			)
 		)
-		(property "Footprint" "Resistor_SMD:R_0805_2012Metric"
+		(property "Footprint" "Resistor_SMD:R_0603_1608Metric_Pad0.98x0.95mm_HandSolder"
 			(at 245.11 132.842 90)
 			(effects
@@
 			)
 		)
-		(property "Footprint" "Resistor_SMD:R_0805_2012Metric"
+		(property "Footprint" "Resistor_SMD:R_0603_1608Metric_Pad0.98x0.95mm_HandSolder"
 			(at 93.218 86.36 90)
 			(effects
@@
 			)
 		)
-		(property "Footprint" "Resistor_SMD:R_0805_2012Metric"
+		(property "Footprint" "Resistor_SMD:R_0603_1608Metric_Pad0.98x0.95mm_HandSolder"
 			(at 93.218 114.3 90)
 			(effects
@@
 			)
 		)
-		(property "Footprint" "Resistor_SMD:R_0805_2012Metric"
+		(property "Footprint" "Resistor_SMD:R_0603_1608Metric_Pad0.98x0.95mm_HandSolder"
 			(at 245.11 149.352 90)
 			(effects
@@
 			)
 		)
-		(property "Footprint" "Resistor_SMD:R_0805_2012Metric"
+		(property "Footprint" "Resistor_SMD:R_0603_1608Metric_Pad0.98x0.95mm_HandSolder"
 			(at 92.71 210.312 90)
 			(effects
@@
 			)
 		)
-		(property "Footprint" "Resistor_SMD:R_0805_2012Metric"
+		(property "Footprint" "Resistor_SMD:R_0603_1608Metric_Pad0.98x0.95mm_HandSolder"
 			(at 184.658 190.5 90)
 			(effects
@@
 			)
 		)
-		(property "Footprint" "Resistor_SMD:R_0805_2012Metric"
+		(property "Footprint" "Resistor_SMD:R_0603_1608Metric_Pad0.98x0.95mm_HandSolder"
 			(at 93.218 58.42 90)
 			(effects
@@
 			)
 		)
-		(property "Footprint" "Resistor_SMD:R_0805_2012Metric"
+		(property "Footprint" "Resistor_SMD:R_0603_1608Metric_Pad0.98x0.95mm_HandSolder"
 			(at 208.28 202.692 90)
 			(effects

Commit message: wip
Parts:
- added C13, C14, C28, C29, C45, C46: C, Capacitor_SMD:C_0603_1608Metric_Pad1.08x0.95mm_HandSolder, symbol Device:C
- added C57, C63: C_Polarized, Capacitor_SMD:CP_Elec_6.3x3, symbol Device:C_Polarized
- added J3: AudioJack2_Ground, TRHMSX:PJ-307, symbol Connector_Audio:AudioJack2_Ground
- added R45, R48, R53, R54, R55, R56, R57, R58, R59, R60, R61, R62, R63, R8: R, Resistor_SMD:R_0603_1608Metric_Pad0.98x0.95mm_HandSolder, symbol Device:R
- added U18: CS4398, Package_SO:TSSOP-28_6.1x9.7mm_P0.65mm, symbol TRHMSX:CS4398
- added U19: NE5532, Package_SO:SOIC-8_3.9x4.9mm_P1.27mm, symbol Amplifier_Operational:NE5532
- renumbered C27 to C10, C26 to C12, C40 to C15, C42 to C16, C41 to C17, C44 to C2, C43 to C3, C39 to C4, C38 to C5, C37 to C6, C36 to C7, C32 to C8, J1 to J2, J16 to J4, J13 to J6, R4 to R1, R25 to R10, R26 to R11, R27 to R12, R28 to R13, R20 to R14, R23 to R2, R6 to R3, R21 to R43, R22 to R44, R18 to R46, R19 to R47, R17 to R49, R15 to R5, R16 to R7, R24 to R9, U12 to U1, U13 to U2, U11 to U3, X1 to X2
Connections:
- net GND: now also C28.2, C29.1, J3.G, R54.1, R55.2
- new net: C14.1, R48.2, R60.1, R61.1
- new net: C14.2, R53.2, R55.1, R57.1
- new net: R48.1, U18.19 (AOUTB-)
- new net: R53.1, U18.20 (AOUTB+)
- new net: R8.1, U18.23 (AOUTA+)
- new net: R45.1, U18.24 (AOUTA-)
- new net: C46.1, R61.2, U19.6 (-)
- new net: C45.2, C57.1, R59.2, U19.1
- new net: C57.2, R62.1
- new net: C13.2, R45.2, R58.1, R59.1
- new net: C29.2, R57.2, U19.5 (+)
- new net: C45.1, R58.2, U19.2 (-)
- new net: C28.1, R56.2, U19.3 (+)
- new net: C46.2, C63.1, R60.2, U19.7
- new net: C63.2, R63.1
- new net: C13.1, R54.2, R56.1, R8.2
- new net +12V: U19.8 (V+)
- new net -12V: U19.4 (V-)
- new net SOUND_L: J3.T, R62.2
- new net SOUND_R: J3.S, R63.2
Other:
- note added: "AUDIO"
- note added: "VIDEO"
